Commit message: feat: visualizing on gazebo, min: gazebo control

File: four_wd_description/urdf/4wd_properties.urdf.xacro (robot description, xacro)
@@ -9,4 +9,6 @@
     <xacro:property name="lidar_radius" value="0.04"/>
     <xacro:property name="lidar_height" value="0.05"/>
+    <!-- Argument -->
+    <xacro:arg name="controller_config_path" default=""/>
     <!-- #################### LINKS #################### -->
     <!-- Base Footprint (at the center of the robot on the ground) -->
@@ -26,5 +28,5 @@
             <origin xyz="0 0 ${base_height/2}" rpy="0 0 0"/>
             <geometry>
-                <box size="${base_length} ${base_width} ${base_height}"/>
+                <box size="${base_length - 0.05} ${base_width} ${base_height - 0.01}"/>
             </geometry>
         </collision>
@@ -110,33 +112,9 @@
     </joint>
     <!-- #################### GAZEBO & ROS2 CONTROL #################### -->
-    <!-- ros2_control Controller Manager -->
-    <ros2_control name="GazeboSystem" type="system">
-        <hardware>
-            <plugin>gazebo_ros2_control/GazeboSystem</plugin>
-        </hardware>
-        <joint name="front_left_wheel_joint">
-            <command_interface name="velocity"/>
-            <state_interface name="position"/>
-            <state_interface name="velocity"/>
-        </joint>
-        <joint name="front_right_wheel_joint">
-            <command_interface name="velocity"/>
-            <state_interface name="position"/>
-            <state_interface name="velocity"/>
-        </joint>
-        <joint name="back_left_wheel_joint">
-            <command_interface name="velocity"/>
-            <state_interface name="position"/>
-            <state_interface name="velocity"/>
-        </joint>
-        <joint name="back_right_wheel_joint">
-            <command_interface name="velocity"/>
-            <state_interface name="position"/>
-            <state_interface name="velocity"/>
-        </joint>
-    </ros2_control>
     <!-- Lidar Sensor Plugin -->
     <gazebo reference="lidar_link">
         <sensor name="gpu_lidar" type="gpu_lidar">
+            <pose>0 0 0 0 0 0</pose>
+            <visualize>true</visualize>
             <topic>/scan</topic>
             <update_rate>10</update_rate>
@@ -146,6 +124,6 @@
                         <samples>360</samples>
                         <resolution>1</resolution>
-                        <min_angle>-3.14</min_angle>
-                        <max_angle>3.14</max_angle>
+                        <min_angle>-3.14159</min_angle>
+                        <max_angle>3.14159</max_angle>
                     </horizontal>
                 </scan>
@@ -153,7 +131,7 @@
                     <min>0.12</min>
                     <max>12.0</max>
+                    <resolution>0.01</resolution>
                 </range>
             </lidar>
-            <visualize>true</visualize>
         </sensor>
     </gazebo>

Commit message: feat: robot moving on gazebo and rviz

File: four_wd_description/urdf/4wd_properties.urdf.xacro (robot description, xacro)
@@ -136,3 +136,36 @@
         </sensor>
     </gazebo>
+    <ros2_control name="GazeboSystem" type="system">
+    <hardware>
+        <plugin>gz_ros2_control/GazeboSimSystem</plugin>
+    </hardware>
+        <joint name="front_left_wheel_joint">
+            <command_interface name="velocity"/>
+            <state_interface name="position"/>
+            <state_interface name="velocity"/>
+        </joint>
+        <joint name="front_right_wheel_joint">
+            <command_interface name="velocity"/>
+            <state_interface name="position"/>
+            <state_interface name="velocity"/>
+        </joint>
+        <joint name="back_left_wheel_joint">
+            <command_interface name="velocity"/>
+            <state_interface name="position"/>
+            <state_interface name="velocity"/>
+        </joint>
+        <joint name="back_right_wheel_joint">
+            <command_interface name="velocity"/>
+            <state_interface name="position"/>
+            <state_interface name="velocity"/>
+        </joint>
+    </ros2_control>
+    <gazebo>
+        <plugin name="gz_ros2_control::GazeboSimROS2ControlPlugin"
+                filename="gz_ros2_control-system">
+            <parameters>$(arg controller_config_path)</parameters>
+            <robot_param>robot_description</robot_param>
+            <robot_param_node>robot_state_publisher</robot_param_node>
+        </plugin>
+    </gazebo>
 </robot>
